File: Hardware/Benchtop Power Supply.brd (EAGLE design)
At the start: 132.1 x 48.3 mm, 24 parts, among them J1 ATX24RH

Commit message: Fixing review commentaries
Other:
- board text added: "ROUTE OUT"
Changed lines of the file:
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@@
 <text x="93.98" y="2.54" size="1.778" layer="21" font="vector" ratio="15">On</text>
 <text x="111.76" y="2.54" size="1.778" layer="21" font="vector" ratio="15">Off</text>
+<text x="6.35" y="36.83" size="1.27" layer="51" font="vector" ratio="15">ROUTE
+OUT</text>
+<text x="25.4" y="36.83" size="1.27" layer="51" font="vector" ratio="15">ROUTE
+OUT</text>
+<text x="38.1" y="35.56" size="1.27" layer="51" font="vector" ratio="15">ROUTE
+OUT</text>
+<text x="57.15" y="36.83" size="1.27" layer="51" font="vector" ratio="15">ROUTE
+OUT</text>
+<text x="69.85" y="36.83" size="1.27" layer="51" font="vector" ratio="15">ROUTE
+OUT</text>
+<text x="88.9" y="36.83" size="1.27" layer="51" font="vector" ratio="15">ROUTE
+OUT</text>
+<text x="101.6" y="35.56" size="1.27" layer="51" font="vector" ratio="15">ROUTE
+OUT</text>
+<text x="120.65" y="36.83" size="1.27" layer="51" font="vector" ratio="15">ROUTE
+OUT</text>
 </plain>
 <attributes>
@@
 <signal name="GND">
 <contactref element="J1" pad="3"/>
-<contactref element="J1" pad="5"/>
-<contactref element="J1" pad="7"/>
-<contactref element="J1" pad="15"/>
-<contactref element="J1" pad="17"/>
-<contactref element="J1" pad="18"/>
-<contactref element="J1" pad="19"/>
-<contactref element="J1" pad="24"/>
 <contactref element="LED1" pad="K"/>
 <polygon width="0.254" layer="16" isolate="0.3048">
@@
 </polygon>
 <contactref element="S9" pad="3"/>
+<contactref element="J1" pad="5"/>
+<contactref element="J1" pad="7"/>
+<contactref element="S3" pad="P$1"/>
+<contactref element="J1" pad="24"/>
+<contactref element="J1" pad="19"/>
 <contactref element="S7" pad="P$1"/>
+<contactref element="J1" pad="18"/>
+<contactref element="S5" pad="P$1"/>
+<contactref element="J1" pad="17"/>
+<contactref element="J1" pad="15"/>
 <contactref element="S1" pad="P$1"/>
-<contactref element="S3" pad="P$1"/>
-<contactref element="S5" pad="P$1"/>
+<wire x1="101.4222" y1="3.81" x2="109.528153125" y2="32.71184375" width="0" layer="19" extent="1-1"/>
+<wire x1="80.74" y1="13.65" x2="101.4222" y2="3.81" width="0" layer="19" extent="1-1"/>
+<wire x1="80.74" y1="19.15" x2="80.74" y2="13.65" width="0" layer="19" extent="1-1"/>
+<wire x1="72.34" y1="19.15" x2="80.74" y2="19.15" width="0" layer="19" extent="1-1"/>
+<wire x1="68.14" y1="19.15" x2="72.34" y2="19.15" width="0" layer="19" extent="1-1"/>
+<wire x1="63.94" y1="19.15" x2="68.14" y2="19.15" width="0" layer="19" extent="1-1"/>
+<wire x1="72.34" y1="13.65" x2="72.34" y2="19.15" width="0" layer="19" extent="1-1"/>
+<wire x1="63.94" y1="13.65" x2="63.94" y2="19.15" width="0" layer="19" extent="1-1"/>
+<wire x1="77.778153125" y1="32.71184375" x2="80.74" y2="19.15" width="0" layer="19" extent="1-1"/>
+<wire x1="42.94" y1="19.15" x2="63.94" y2="19.15" width="0" layer="19" extent="1-1"/>
+<wire x1="46.028153125" y1="32.71184375" x2="42.94" y2="19.15" width="0" layer="19" extent="1-1"/>
+<wire x1="27.94" y1="5.08" x2="42.94" y2="19.15" width="0" layer="19" extent="1-1"/>
+<wire x1="14.278153125" y1="32.71184375" x2="27.94" y2="5.08" width="0" layer="19" extent="1-1"/>
 </signal>
 <signal name="5V">
@@
 </board>
 </drawing>
+<compatibility>
+<note version="6.3" minversion="6.2.2" severity="warning">
+Since Version 6.2.2 text objects can contain more than one line,
+which will not be processed correctly with this version.
+</note>
+</compatibility>
 </eagle>
