File: Hardware/Benchtop Power Supply.sch (EAGLE design)
At the start: 20 parts, among them J1 ATX24RH

Commit message: Midway hardware changes
Parts:
- added FRAME1: FRAME-LETTER, SparkFun-Aesthetics:FRAME-LETTER
- added S9: (no value), SparkFun-Electromechanical:SWITCH-SPDTKIT
- added U$1: REVISION, SparkFun-Aesthetics:REVISION
- J1: device SparkFun:ATX24RH -> SparkFun-Connectors:ATX24RH
Connections:
- new net N$2: J1.PS_ON, S9.P
- net GND: now also S9.S; no longer J1.PS_ON
Other:
- note added: "Ryan Owens"
- note added: "Toni Klopfenstein"
- note added: "v1.3"
Changed lines of the file:
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@@
 <layer number="106" name="bPlate" color="7" fill="1" visible="yes" active="yes"/>
 <layer number="107" name="Crop" color="7" fill="1" visible="yes" active="yes"/>
+<layer number="108" name="tplace-old" color="10" fill="1" visible="yes" active="yes"/>
+<layer number="109" name="ref-old" color="11" fill="1" visible="yes" active="yes"/>
+<layer number="110" name="fp0" color="7" fill="1" visible="yes" active="yes"/>
+<layer number="111" name="LPC17xx" color="7" fill="1" visible="yes" active="yes"/>
+<layer number="112" name="tSilk" color="7" fill="1" visible="yes" active="yes"/>
+<layer number="113" name="IDFDebug" color="4" fill="1" visible="yes" active="yes"/>
 <layer number="116" name="Patch_BOT" color="9" fill="4" visible="yes" active="yes"/>
 <layer number="121" name="_tsilk" color="7" fill="1" visible="yes" active="yes"/>
 <layer number="122" name="_bsilk" color="7" fill="1" visible="yes" active="yes"/>
+<layer number="123" name="tTestmark" color="7" fill="1" visible="yes" active="yes"/>
+<layer number="124" name="bTestmark" color="7" fill="1" visible="yes" active="yes"/>
+<layer number="125" name="_tNames" color="7" fill="1" visible="yes" active="yes"/>
+<layer number="126" name="_bNames" color="7" fill="1" visible="yes" active="yes"/>
+<layer number="127" name="_tValues" color="7" fill="1" visible="yes" active="yes"/>
+<layer number="128" name="_bValues" color="7" fill="1" visible="yes" active="yes"/>
+<layer number="131" name="tAdjust" color="7" fill="1" visible="yes" active="yes"/>
+<layer number="132" name="bAdjust" color="7" fill="1" visible="yes" active="yes"/>
+<layer number="144" name="Drill_legend" color="7" fill="1" visible="yes" active="yes"/>
 <layer number="151" name="HeatSink" color="7" fill="1" visible="yes" active="yes"/>
+<layer number="152" name="_bDocu" color="7" fill="1" visible="yes" active="yes"/>
+<layer number="199" name="Contour" color="7" fill="1" visible="yes" active="yes"/>
 <layer number="200" name="200bmp" color="1" fill="10" visible="yes" active="yes"/>
 <layer number="201" name="201bmp" color="2" fill="10" visible="yes" active="yes"/>
@@
 <layer number="207" name="207bmp" color="8" fill="10" visible="yes" active="yes"/>
 <layer number="208" name="208bmp" color="9" fill="10" visible="yes" active="yes"/>
+<layer number="209" name="209bmp" color="7" fill="1" visible="yes" active="yes"/>
+<layer number="210" name="210bmp" color="7" fill="1" visible="yes" active="yes"/>
+<layer number="211" name="211bmp" color="7" fill="1" visible="yes" active="yes"/>
+<layer number="212" name="212bmp" color="7" fill="1" visible="yes" active="yes"/>
+<layer number="213" name="213bmp" color="7" fill="1" visible="yes" active="yes"/>
+<layer number="214" name="214bmp" color="7" fill="1" visible="yes" active="yes"/>
+<layer number="215" name="215bmp" color="7" fill="1" visible="yes" active="yes"/>
+<layer number="216" name="216bmp" color="7" fill="1" visible="yes" active="yes"/>
+<layer number="217" name="217bmp" color="18" fill="1" visible="no" active="no"/>
+<layer number="218" name="218bmp" color="19" fill="1" visible="no" active="no"/>
+<layer number="219" name="219bmp" color="20" fill="1" visible="no" active="no"/>
+<layer number="220" name="220bmp" color="21" fill="1" visible="no" active="no"/>
+<layer number="221" name="221bmp" color="22" fill="1" visible="no" active="no"/>
+<layer number="222" name="222bmp" color="23" fill="1" visible="no" active="no"/>
+<layer number="223" name="223bmp" color="24" fill="1" visible="no" active="no"/>
+<layer number="224" name="224bmp" color="25" fill="1" visible="no" active="no"/>
+<layer number="248" name="Housing" color="7" fill="1" visible="yes" active="yes"/>
+<layer number="249" name="Edge" color="7" fill="1" visible="yes" active="yes"/>
 <layer number="250" name="Descript" color="3" fill="1" visible="no" active="no"/>
 <layer number="251" name="SMDround" color="12" fill="11" visible="no" active="no"/>
@@
 </classes>
 <parts>
-<part name="FRAME1" library="SparkFun" deviceset="FRAME-LETTER" device=""/>
+<part name="FRAME1" library="SparkFun-Aesthetics" deviceset="FRAME-LETTER" device=""/>
 <part name="JP1" library="SparkFun" deviceset="LOGO-SFE" device="NEW"/>
 <part name="JP2" library="SparkFun" deviceset="STAND-OFF" device=""/>
@@
 <part name="JP4" library="SparkFun" deviceset="STAND-OFF" device=""/>
 <part name="JP5" library="SparkFun" deviceset="STAND-OFF" device=""/>
-<part name="J1" library="SparkFun" deviceset="ATX24" device="RH"/>
+<part name="J1" library="SparkFun-Connectors" deviceset="ATX24" device="RH"/>
 <part name="GND1" library="SparkFun" deviceset="GND" device=""/>
 <part name="GND2" library="SparkFun" deviceset="GND" device=""/>
@@
 <part name="S7" library="SparkFun" deviceset="BINDING_POST" device=""/>
 <part name="S8" library="SparkFun" deviceset="BINDING_POST" device=""/>
+<part name="S9" library="SparkFun-Electromechanical" deviceset="SWITCH-SPDT" device="KIT"/>
+<part name="U$1" library="SparkFun-Aesthetics" deviceset="REVISION" device=""/>
 </parts>
 <sheets>
 <sheet>
 <plain>
+<text x="171.704" y="11.938" size="2.54" layer="94">Ryan Owens</text>
+<text x="175.26" y="7.62" size="2.54" layer="94">Toni Klopfenstein</text>
+<text x="238.76" y="7.62" size="2.54" layer="94">v1.3</text>
 </plain>
 <instances>
 <instance part="FRAME1" gate="G$1" x="0" y="0"/>
 <instance part="FRAME1" gate="G$2" x="147.32" y="0"/>
-<instance part="JP1" gate="G$1" x="152.4" y="27.94"/>
-<instance part="JP2" gate="G$1" x="162.56" y="33.02"/>
-<instance part="JP3" gate="G$1" x="162.56" y="25.4"/>
-<instance part="JP4" gate="G$1" x="167.64" y="33.02"/>
-<instance part="JP5" gate="G$1" x="167.64" y="25.4"/>
+<instance part="JP1" gate="G$1" x="241.3" y="17.78"/>
+<instance part="JP2" gate="G$1" x="246.38" y="33.02"/>
+<instance part="JP3" gate="G$1" x="241.3" y="25.4"/>
+<instance part="JP4" gate="G$1" x="241.3" y="33.02"/>
+<instance part="JP5" gate="G$1" x="246.38" y="25.4"/>
 <instance part="J1" gate="G$1" x="121.92" y="104.14"/>
 <instance part="GND1" gate="1" x="104.14" y="78.74"/>
-<instance part="GND2" gate="1" x="137.16" y="78.74"/>
+<instance part="GND2" gate="1" x="149.86" y="78.74"/>
 <instance part="F1" gate="G$1" x="76.2" y="121.92"/>
 <instance part="F2" gate="G$1" x="165.1" y="121.92"/>
@@
 <instance part="S7" gate="G$1" x="53.34" y="121.92"/>
 <instance part="S8" gate="G$1" x="48.26" y="121.92"/>
+<instance part="S9" gate="1" x="142.24" y="91.44"/>
+<instance part="U$1" gate="G$1" x="148.59" y="7.112"/>
 </instances>
 <busses>
@@
 <nets>
 <net name="GND" class="0">
-<segment>
-<wire x1="134.62" y1="91.44" x2="137.16" y2="91.44" width="0.1524" layer="91"/>
-<wire x1="137.16" y1="91.44" x2="137.16" y2="81.28" width="0.1524" layer="91"/>
-<pinref part="J1" gate="G$1" pin="PS_ON"/>
-<pinref part="GND2" gate="1" pin="GND"/>
-</segment>
 <segment>
 <wire x1="106.68" y1="83.82" x2="104.14" y2="83.82" width="0.1524" layer="91"/>
@@
 <pinref part="LED1" gate="G$1" pin="C"/>
 </segment>
+<segment>
+<pinref part="S9" gate="1" pin="S"/>
+<wire x1="147.32" y1="88.9" x2="149.86" y2="88.9" width="0.2032" layer="91"/>
+<wire x1="149.86" y1="88.9" x2="149.86" y2="81.28" width="0.2032" layer="91"/>
+<pinref part="GND2" gate="1" pin="GND"/>
+</segment>
 </net>
 <net name="5V" class="0">
@@
 </segment>
 </net>
+<net name="N$2" class="0">
+<segment>
+<pinref part="J1" gate="G$1" pin="PS_ON"/>
+<pinref part="S9" gate="1" pin="P"/>
+<wire x1="134.62" y1="91.44" x2="139.7" y2="91.44" width="0.2032" layer="91"/>
+</segment>
+</net>

Commit message: Files changed for V13- ready for review
Parts:
- added LOGO1: OSHW-LOGOL, SparkFun-Aesthetics:OSHW-LOGOL
- JP1: value LOGO-SFENEW -> SFE_LOGO_NAME_FLAME.3_INCH; device SparkFun:LOGO-SFENEW -> SparkFun-Aesthetics:SFE_LOGO_NAME_FLAME.3_INCH
Connections:
- new net NC: S9.O
Changed lines of the file:
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@@
 <parts>
 <part name="FRAME1" library="SparkFun-Aesthetics" deviceset="FRAME-LETTER" device=""/>
-<part name="JP1" library="SparkFun" deviceset="LOGO-SFE" device="NEW"/>
+<part name="JP1" library="SparkFun-Aesthetics" deviceset="SFE_LOGO_NAME_FLAME" device=".3_INCH" value="SFE_LOGO_NAME_FLAME.3_INCH"/>
 <part name="JP2" library="SparkFun" deviceset="STAND-OFF" device=""/>
 <part name="JP3" library="SparkFun" deviceset="STAND-OFF" device=""/>
@@
 <part name="S9" library="SparkFun-Electromechanical" deviceset="SWITCH-SPDT" device="KIT"/>
 <part name="U$1" library="SparkFun-Aesthetics" deviceset="REVISION" device=""/>
+<part name="LOGO1" library="SparkFun-Aesthetics" deviceset="OSHW-LOGO" device="L"/>
 </parts>
 <sheets>
@@
 <instance part="FRAME1" gate="G$1" x="0" y="0"/>
 <instance part="FRAME1" gate="G$2" x="147.32" y="0"/>
-<instance part="JP1" gate="G$1" x="241.3" y="17.78"/>
+<instance part="JP1" gate="G$1" x="91.44" y="0"/>
 <instance part="JP2" gate="G$1" x="246.38" y="33.02"/>
 <instance part="JP3" gate="G$1" x="241.3" y="25.4"/>
@@
 <instance part="LED1" gate="G$1" x="91.44" y="104.14"/>
 <instance part="GND3" gate="1" x="91.44" y="93.98"/>
-<instance part="S1" gate="G$1" x="198.12" y="121.92"/>
-<instance part="S2" gate="G$1" x="203.2" y="121.92"/>
-<instance part="S3" gate="G$1" x="198.12" y="104.14"/>
-<instance part="S4" gate="G$1" x="203.2" y="104.14"/>
-<instance part="S5" gate="G$1" x="198.12" y="96.52"/>
-<instance part="S6" gate="G$1" x="203.2" y="96.52"/>
-<instance part="S7" gate="G$1" x="53.34" y="121.92"/>
-<instance part="S8" gate="G$1" x="48.26" y="121.92"/>
+<instance part="S1" gate="G$1" x="208.28" y="121.92"/>
+<instance part="S2" gate="G$1" x="213.36" y="121.92"/>
+<instance part="S3" gate="G$1" x="208.28" y="104.14"/>
+<instance part="S4" gate="G$1" x="213.36" y="104.14"/>
+<instance part="S5" gate="G$1" x="208.28" y="96.52"/>
+<instance part="S6" gate="G$1" x="213.36" y="96.52"/>
+<instance part="S7" gate="G$1" x="43.18" y="121.92"/>
+<instance part="S8" gate="G$1" x="38.1" y="121.92"/>
 <instance part="S9" gate="1" x="142.24" y="91.44"/>
 <instance part="U$1" gate="G$1" x="148.59" y="7.112"/>
+<instance part="LOGO1" gate="G$1" x="76.2" y="10.16"/>
 </instances>
 <busses>
@@
 <segment>
 <pinref part="S9" gate="1" pin="S"/>
-<wire x1="147.32" y1="88.9" x2="149.86" y2="88.9" width="0.2032" layer="91"/>
-<wire x1="149.86" y1="88.9" x2="149.86" y2="81.28" width="0.2032" layer="91"/>
+<wire x1="147.32" y1="88.9" x2="149.86" y2="88.9" width="0.127" layer="91"/>
+<wire x1="149.86" y1="88.9" x2="149.86" y2="81.28" width="0.127" layer="91"/>
 <pinref part="GND2" gate="1" pin="GND"/>
 </segment>
@@
 <segment>
 <wire x1="66.04" y1="121.92" x2="58.42" y2="121.92" width="0.1524" layer="91"/>
-<label x="58.42" y="121.92" size="1.778" layer="95"/>
 <pinref part="F1" gate="G$1" pin="1"/>
+<label x="58.42" y="121.92" size="1.778" layer="95" rot="R180" xref="yes"/>
 </segment>
 </net>
@@
 <segment>
 <wire x1="175.26" y1="121.92" x2="190.5" y2="121.92" width="0.1524" layer="91"/>
-<label x="185.42" y="121.92" size="1.778" layer="95"/>
 <pinref part="F2" gate="G$1" pin="2"/>
+<label x="190.5" y="121.92" size="1.778" layer="95" xref="yes"/>
 </segment>
 </net>
@@
 <segment>
 <wire x1="175.26" y1="104.14" x2="190.5" y2="104.14" width="0.1524" layer="91"/>
-<label x="185.42" y="104.14" size="1.778" layer="95"/>
 <pinref part="F3" gate="G$1" pin="2"/>
+<label x="190.5" y="104.14" size="1.778" layer="95" xref="yes"/>
 </segment>
 </net>
@@
 <segment>
 <wire x1="175.26" y1="96.52" x2="190.5" y2="96.52" width="0.1524" layer="91"/>
-<label x="185.42" y="96.52" size="1.778" layer="95"/>
 <pinref part="F4" gate="G$1" pin="2"/>
+<label x="190.5" y="96.52" size="1.778" layer="95" xref="yes"/>
 </segment>
 </net>
@@
 <pinref part="J1" gate="G$1" pin="PS_ON"/>
 <pinref part="S9" gate="1" pin="P"/>
-<wire x1="134.62" y1="91.44" x2="139.7" y2="91.44" width="0.2032" layer="91"/>
-</segment>
-</net>
+<wire x1="134.62" y1="91.44" x2="139.7" y2="91.44" width="0.127" layer="91"/>
+</segment>
+</net>
+<net name="NC" class="0">
+<segment>
+<pinref part="S9" gate="1" pin="O"/>
+<wire x1="147.32" y1="93.98" x2="152.4" y2="93.98" width="0.127" layer="91"/>
+<label x="152.4" y="93.98" size="1.778" layer="95" xref="yes"/>
+</segment>
+</net>

Commit message: Adding rounded corners, square binding post holes, increased traces to 60 mil
Parts:
- S1, S2, S3, S4, S5, S6, S7, S8: device SparkFun:BINDING_POST -> SparkFun-Connectors:BINDING_POST
Changed lines of the file:
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@@
 <part name="LED1" library="SparkFun" deviceset="LED" device="5MM" value="RED"/>
 <part name="GND3" library="SparkFun" deviceset="GND" device=""/>
-<part name="S1" library="SparkFun" deviceset="BINDING_POST" device=""/>
-<part name="S2" library="SparkFun" deviceset="BINDING_POST" device=""/>
-<part name="S3" library="SparkFun" deviceset="BINDING_POST" device=""/>
-<part name="S4" library="SparkFun" deviceset="BINDING_POST" device=""/>
-<part name="S5" library="SparkFun" deviceset="BINDING_POST" device=""/>
-<part name="S6" library="SparkFun" deviceset="BINDING_POST" device=""/>
-<part name="S7" library="SparkFun" deviceset="BINDING_POST" device=""/>
-<part name="S8" library="SparkFun" deviceset="BINDING_POST" device=""/>
+<part name="S1" library="SparkFun-Connectors" deviceset="BINDING_POST" device=""/>
+<part name="S2" library="SparkFun-Connectors" deviceset="BINDING_POST" device=""/>
+<part name="S3" library="SparkFun-Connectors" deviceset="BINDING_POST" device=""/>
+<part name="S4" library="SparkFun-Connectors" deviceset="BINDING_POST" device=""/>
+<part name="S5" library="SparkFun-Connectors" deviceset="BINDING_POST" device=""/>
+<part name="S6" library="SparkFun-Connectors" deviceset="BINDING_POST" device=""/>
+<part name="S7" library="SparkFun-Connectors" deviceset="BINDING_POST" device=""/>
+<part name="S8" library="SparkFun-Connectors" deviceset="BINDING_POST" device=""/>
 <part name="S9" library="SparkFun-Electromechanical" deviceset="SWITCH-SPDT" device="KIT"/>
 <part name="U$1" library="SparkFun-Aesthetics" deviceset="REVISION" device=""/>

Commit message: Fixing drill holes for mounting posts
Parts:
- JP2, JP3, JP4, JP5: device SparkFun:STAND-OFF -> SparkFun-Electromechanical:STAND-OFF
Changed lines of the file:
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@@
 <layer number="54" name="bGND_GNDA" color="1" fill="9" visible="no" active="no"/>
 <layer number="56" name="wert" color="7" fill="1" visible="no" active="no"/>
+<layer number="57" name="tCAD" color="7" fill="1" visible="no" active="no"/>
 <layer number="91" name="Nets" color="2" fill="1" visible="yes" active="yes"/>
 <layer number="92" name="Busses" color="1" fill="1" visible="yes" active="yes"/>
@@
 <layer number="97" name="Info" color="7" fill="1" visible="yes" active="yes"/>
 <layer number="98" name="Guide" color="6" fill="1" visible="yes" active="yes"/>
+<layer number="99" name="SpiceOrder" color="7" fill="1" visible="yes" active="yes"/>
 <layer number="100" name="Muster" color="7" fill="1" visible="no" active="no"/>
 <layer number="101" name="Patch_Top" color="12" fill="4" visible="yes" active="yes"/>
@@
 <layer number="132" name="bAdjust" color="7" fill="1" visible="yes" active="yes"/>
 <layer number="144" name="Drill_legend" color="7" fill="1" visible="yes" active="yes"/>
+<layer number="150" name="Notes" color="7" fill="1" visible="yes" active="yes"/>
 <layer number="151" name="HeatSink" color="7" fill="1" visible="yes" active="yes"/>
 <layer number="152" name="_bDocu" color="7" fill="1" visible="yes" active="yes"/>
+<layer number="153" name="FabDoc1" color="7" fill="1" visible="yes" active="yes"/>
+<layer number="154" name="FabDoc2" color="7" fill="1" visible="yes" active="yes"/>
+<layer number="155" name="FabDoc3" color="7" fill="1" visible="yes" active="yes"/>
 <layer number="199" name="Contour" color="7" fill="1" visible="yes" active="yes"/>
 <layer number="200" name="200bmp" color="1" fill="10" visible="yes" active="yes"/>
@@
 <part name="FRAME1" library="SparkFun-Aesthetics" deviceset="FRAME-LETTER" device=""/>
 <part name="JP1" library="SparkFun-Aesthetics" deviceset="SFE_LOGO_NAME_FLAME" device=".3_INCH" value="SFE_LOGO_NAME_FLAME.3_INCH"/>
-<part name="JP2" library="SparkFun" deviceset="STAND-OFF" device=""/>
-<part name="JP3" library="SparkFun" deviceset="STAND-OFF" device=""/>
-<part name="JP4" library="SparkFun" deviceset="STAND-OFF" device=""/>
-<part name="JP5" library="SparkFun" deviceset="STAND-OFF" device=""/>
+<part name="JP2" library="SparkFun-Electromechanical" deviceset="STAND-OFF" device=""/>
+<part name="JP3" library="SparkFun-Electromechanical" deviceset="STAND-OFF" device=""/>
+<part name="JP4" library="SparkFun-Electromechanical" deviceset="STAND-OFF" device=""/>
+<part name="JP5" library="SparkFun-Electromechanical" deviceset="STAND-OFF" device=""/>
 <part name="J1" library="SparkFun-Connectors" deviceset="ATX24" device="RH"/>
 <part name="GND1" library="SparkFun" deviceset="GND" device=""/>
